File: Uni60/UNI60_Solder/Uni60_Solder_KiCad/Uni60_Solder.kicad_pcb (KiCad board)
At the start: 2 copper layers, 284.7 x 94.2 mm, 202 parts, among them J1 Conn_01x04, J2 Conn_01x04, J3 Conn_01x04, J4 Conn_01x04, J5 Conn_01x04, J6 Conn_01x04, SW1 SW_Push, SW2 SW_Push, U1 STM32F072CBTx, U2 XC6206PxxxMR, U3 USBLC6-2SC6

Commit message: updated traces
Routing:
- net /COL1: track 123.4 -> 116.0 mm
- net +5V: track 160.8 -> 153.6 mm
- net /USB_D-: track 148.1 -> 141.2 mm
- net /USB_D+: track 145.8 -> 139.2 mm
- net GND: vias 41 -> 43

Commit message: added molex connector to my library
Parts:
- J6: footprint Connector_Molex:Molex_Pico-EZmate_78171-0004_1x04-1MP_P1.20mm_Vertical -> shentobento:Molex_Pico-EZmate_78171-0004_1x04-1MP_P1.20mm_Vertical
Other:
- board text added: "For Instructional Use Only."
- board text added: "SOLIDWORKS Educational Product."

Commit message: idk
Routing:
- net /COL11: track 290.3 -> 291.0 mm
- net GND: vias 43 -> 46
Other:
- board text added: "Uni60 v1.0 by ShentoBento github.com/ShentoBento/Universal_PCBs"
- board text removed: "Uni60 v1.0 by ShentoBento"
