File: Uni60/UNI60_Solder/Uni60_Solder_KiCad/Uni60_Solder.kicad_sch (KiCad schematic)
At the start: 193 parts, among them J1 Conn_01x04, J2 Conn_01x04, J3 Conn_01x04, J4 Conn_01x04, J5 Conn_01x04, J6 Conn_01x04, J7 USB_C_Receptacle_USB2.0_14P, SW1 SW_Push, SW2 SW_Push, U1 STM32F072CBTx, U2 XC6206PxxxMR, U3 USBLC6-2SC6

Commit message: added alps-mx footprints
Parts:
- KC_0, KC_1, KC_2, KC_3, KC_4, KC_5, KC_6, KC_7, KC_8, KC_9, KC_<>1, KC_A1, KC_B1, KC_BKSP1, KC_BKSP2, KC_BSLS2, KC_BSLS_ISO1, KC_C1, KC_COMM1, KC_D1, KC_DOT1, KC_E1, KC_ENT1, KC_ENT_ISO1, KC_EQL1, KC_ESC1, KC_F1, KC_G1, KC_H1, KC_I1, KC_J1, KC_K1, KC_L1, KC_LBRC1, KC_LGUI1, KC_LSFT1, KC_M1, KC_MINS1, KC_MO1, KC_N1, KC_O1, KC_P1, KC_Q1, KC_QUOT1, KC_R1, KC_RBRC1, KC_RGUI1, KC_RSFT1, KC_RSFT_2.75u1, KC_S1, KC_SCLN1, KC_SLSH1, KC_SPC1, KC_SPC_2.75U1, KC_SPC_3U1, KC_SPC_6.25U1, KC_SPLIT_SPC_2.25U1, KC_SPLIT_SPC_3U1, KC_T1, KC_U1, KC_V1, KC_W1, KC_X1, KC_Y1, KC_Z1: footprint shentobento:SW_MX_1u -> shentobento:SW_Alps_MX_1u
- KC_BSLS1, KC_LCTL1, KC_RALT1, KC_TAB1: footprint shentobento:SW_MX_1.5u -> shentobento:SW_Alps_MX_1.5u
- KC_CAPS1: footprint shentobento:SW_MX_1.75u -> shentobento:SW_Alps_MX_1.75u
- KC_LALT1, KC_RCTL1: footprint shentobento:SW_MX_1.5u -> shentobento:SW_Alps_MX_1u
- KC_LALT_1.25U1, KC_LCTL_1.25U1, KC_LGUI_1.25U1, KC_LSFT2, KC_MENU1, KC_RALT_1.25U1, KC_RCTL_1.25U1, KC_RGUI_1.25U1, KC_SPLIT_FN_1.25U1: footprint shentobento:SW_MX_1.25u -> shentobento:SW_Alps_MX_1.25u
- KC_STEP1: footprint shentobento:SW_MX_1.75u_STEPPED_1.25 -> shentobento:SW_Alps_MX_1.75u_STP_1.25
Connections:
- net COL0: now also KC_STEP1.2; no longer KC_STEP1.1
- net COL6: now also KC_SPLIT_FN_1.25U1.2; no longer KC_SPLIT_FN_1.25U1.1
- net at D29.2 (A), KC_CAPS1.2: now also KC_STEP1.1; no longer KC_STEP1.2
- net at D59.2 (A), KC_SPC1.2, KC_SPC_6.25U1.2: now also KC_SPLIT_FN_1.25U1.1; no longer KC_SPLIT_FN_1.25U1.2
Other:
- moved on the sheet: KC_SPLIT_FN_1.25U1, KC_STEP1
