File: Uni60/UNI60_Hotswap/Uni60_Hotswap_KiCad/Uni60_Hotswap.kicad_pcb (KiCad board)
At the start: 2 copper layers, 284.7 x 94.2 mm, 202 parts, among them J1 Conn_01x04, J2 Conn_01x04, J3 Conn_01x04, J4 Conn_01x04, J5 Conn_01x04, J6 Conn_01x04, SW1 SW_Push, SW2 SW_Push, U1 STM32F072CBTx, U2 XC6206PxxxMR, U3 USBLC6-2SC6

Commit message: changed solder to hotswap sockets
Parts:
- removed KC_SPC_3U1, KC_SPLIT_SPC_3U1: MX_SW_solder, shentobento:SW_MX_1u
- removed the REF** at (214.3, 154.6)
- removed the REF** at (176.2, 154.6)
- removed the REF** at (252.4, 154.6)
- KC_0, KC_1, KC_2, KC_3, KC_4, KC_5, KC_6, KC_7, KC_8, KC_9, KC_<>1, KC_A1, KC_B1, KC_BKSP1, KC_BKSP2, KC_BSLS2, KC_BSLS_ISO1, KC_C1, KC_COMM1, KC_D1, KC_DOT1, KC_E1, KC_ENT1, KC_ENT_ISO1, KC_EQL1, KC_ESC1, KC_F1, KC_G1, KC_H1, KC_I1, KC_J1, KC_K1, KC_L1, KC_LBRC1, KC_LGUI1, KC_LSFT1, KC_M1, KC_MINS1, KC_MO1, KC_N1, KC_O1, KC_P1, KC_Q1, KC_QUOT1, KC_R1, KC_RBRC1, KC_RGUI1, KC_RSFT1, KC_RSFT_2.75u1, KC_S1, KC_SCLN1, KC_SLSH1, KC_SPC1, KC_SPC_2.75U1, KC_SPC_6.25U1, KC_SPLIT_SPC_2.25U1, KC_T1, KC_U1, KC_V1, KC_W1, KC_X1, KC_Y1, KC_Z1: footprint shentobento:SW_MX_1u -> shentobento:SW_MX_HS_KAILH_1u; moved to B.Cu
- KC_BSLS1, KC_LALT1, KC_LCTL1, KC_RALT1, KC_RCTL1, KC_TAB1: footprint shentobento:SW_MX_1.5u -> shentobento:SW_MX_HS_KAILH_1.5u; moved to B.Cu
- KC_CAPS1: footprint shentobento:SW_MX_1.75u -> shentobento:SW_MX_HS_KAILH_1.75u; moved to B.Cu
- KC_LALT_1.25U1, KC_LCTL_1.25U1, KC_LGUI_1.25U1, KC_LSFT2, KC_MENU1, KC_RALT_1.25U1, KC_RCTL_1.25U1, KC_RGUI_1.25U1, KC_SPLIT_FN_1.25U1: footprint shentobento:SW_MX_1.25u -> shentobento:SW_MX_HS_KAILH_1.25u; moved to B.Cu
- KC_STEP1: footprint shentobento:SW_MX_1.75u_STEPPED_1.25 -> shentobento:SW_MX_HS_KAILH_1.75u_STEPPED_1.25; moved to B.Cu
- moved D14 22.0 mm to (319.4, 78.4)
- moved D42 13.8 mm to (338.1, 86.8), turned to 0 degrees
- moved D11 11.3 mm to (264.0, 78.4), turned to -90 degrees
- moved D10 11.3 mm to (245.0, 78.4), turned to -90 degrees
- moved D3 11.2 mm to (111.6, 78.4), turned to -90 degrees
- moved D12 11.0 mm to (283.4, 78.4), turned to -90 degrees
- moved D6 5.34 mm to (183.7, 78.4)
- moved D7 5.34 mm to (202.7, 78.4)
- moved D8 5.34 mm to (221.8, 78.4)
- moved D9 5.34 mm to (240.8, 78.4)
- moved D13 5.34 mm to (317.0, 78.4)
- moved D2 5.12 mm to (107.2, 78.4)
- moved D4 5.12 mm to (145.3, 78.4)
- moved D1 4.64 mm to (83.9, 86.5), turned to 180 degrees
- moved D5 0.80 mm to (164.3, 78.4)
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Routing:
- net /COL13: track 366.0 -> 0.00 mm, vias 2 -> 0
- net /ROW4: track 329.6 -> 7.50 mm, vias 2 -> 0
- net /ROW0: track 306.8 -> 0.00 mm, vias 6 -> 0
- net /COL6: track 220.3 -> 0.00 mm
- net /COL3: track 161.7 -> 0.00 mm, vias 2 -> 0
- net /COL5: track 160.0 -> 0.00 mm
- net /COL4: track 145.4 -> 0.00 mm
- net /COL7: track 244.5 -> 120.3 mm
- net /COL12: track 354.4 -> 234.5 mm
- net /COL0: track 123.2 -> 12.7 mm
- net /COL11: track 290.5 -> 188.3 mm
- net /COL10: track 271.8 -> 170.6 mm
- net /ROW2: track 321.3 -> 236.2 mm, vias 6 -> 2
- net /COL9: track 231.4 -> 153.0 mm
- net /COL8: track 212.8 -> 135.2 mm
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
Commit message: wiring up sockets
Parts:
- moved C3 14.9 mm to (91.1, 105.5)
- moved C7 11.1 mm to (110.4, 105.5)
- moved C8 11.1 mm to (105.5, 104.1)
- moved U2 11.1 mm to (108.6, 104.6)
- moved C1 6.87 mm to (104.8, 106.1), turned to -45 degrees
- moved C9 6.33 mm to (94.1, 112.1), turned to -135 degrees
- moved D43 5.52 mm to (96.4, 144.5)
- moved D54 5.35 mm to (333.1, 144.2)
- moved D29 4.49 mm to (92.9, 124.3)
- moved C2 2.66 mm to (96.7, 101.6), turned to 45 degrees
- moved U1 1.60 mm to (98.5, 107.9), turned to 45 degrees
- moved C4 1.52 mm to (100.3, 114.1), turned to -135 degrees
- moved C6 1.49 mm to (94.7, 101.6), turned to -135 degrees
- turned KC_<>1 to 180 degrees
- turned KC_BSLS1 to 90 degrees
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Routing:
- net /ROW3: track 254.7 -> 0.00 mm
- net /ROW1: track 248.4 -> 0.00 mm, vias 2 -> 0
- net /ROW2: track 236.2 -> 0.00 mm, vias 2 -> 0
- net /COL13: track 0.00 -> 137.5 mm, vias 0 -> 2
- net /COL12: track 234.5 -> 122.8 mm
- net /COL11: track 188.3 -> 79.2 mm
- net /COL6: track 0.00 -> 105.1 mm
- net /COL3: track 0.00 -> 100.1 mm
- net /COL9: track 153.0 -> 59.5 mm
- net /COL10: track 170.6 -> 81.2 mm
- net /COL0: track 12.7 -> 93.2 mm
- net +5V: track 153.2 -> 79.5 mm, vias 5 -> 0
- net /COL4: track 0.00 -> 67.7 mm
- net /COL5: track 0.00 -> 67.7 mm
- net /COL8: track 135.2 -> 67.7 mm
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
Commit message: final changes
Parts:
- moved D29 14.8 mm to (78.6, 120.4), turned to -90 degrees
- moved D41 11.4 mm to (331.0, 125.5), turned to 180 degrees
- moved D70 11.0 mm to (173.2, 151.9), turned to -90 degrees
- moved D59 5.53 mm to (221.5, 154.0)
- moved D58 4.77 mm to (140.2, 149.9), turned to -90 degrees
- moved D57 4.48 mm to (116.4, 150.2), turned to -90 degrees
- moved D56 4.48 mm to (92.6, 150.2), turned to -90 degrees
Routing:
- net Net-(D55-A): track 6.05 -> 0.00 mm
- net Net-(D53-A): track 6.05 -> 0.00 mm
- net Net-(D52-A): track 6.05 -> 0.00 mm
- net Net-(D51-A): track 6.05 -> 0.00 mm
- net Net-(D50-A): track 6.05 -> 0.00 mm
- net Net-(D49-A): track 6.05 -> 0.00 mm
- net Net-(D48-A): track 6.05 -> 0.00 mm
- net Net-(D47-A): track 6.05 -> 0.00 mm
- net Net-(D46-A): track 6.05 -> 0.00 mm
- net Net-(D45-A): track 6.05 -> 0.00 mm
- net Net-(D44-A): track 6.05 -> 0.00 mm
- net Net-(D40-A): track 6.05 -> 0.00 mm
- net Net-(D39-A): track 6.05 -> 0.00 mm
- net Net-(D38-A): track 6.05 -> 0.00 mm
- net Net-(D37-A): track 6.05 -> 0.00 mm
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