File: Uni60/UNI60_Hotswap/Uni60_Hotswap_KiCad/Uni60_Hotswap.kicad_pcb (KiCad board)
At the start: 2 copper layers, 284.7 x 94.2 mm, 197 parts, among them J1 Conn_01x04, J2 Conn_01x04, J3 Conn_01x04, J4 Conn_01x04, J5 Conn_01x04, J6 Conn_01x04, SW1 SW_Push, SW2 SW_Push, U1 STM32F072CBTx, U2 XC6206PxxxMR, U3 USBLC6-2SC6

Commit message: idk
Parts:
- D1, D10, D11, D12, D13, D14, D15, D16, D17, D18, D19, D2, D20, D21, D22, D23, D24, D25, D26, D27, D28, D29, D3, D30, D31, D32, D33, D34, D35, D36, D37, D38, D39, D4, D40, D41, D42, D43, D44, D45, D46, D47, D48, D49, D5, D50, D51, D52, D53, D54, D55, D56, D57, D58, D59, D6, D60, D61, D62, D63, D64, D65, D66, D67, D68, D69, D7, D70, D72, D73, D8, D9: footprint shentobento:D_SOD-123 -> Diode_SMD:D_SOD-323
- moved D65 126.3 mm to (187.2, 156.4)
- moved D63 126.3 mm to (180.1, 156.4)
- moved D64 126.3 mm to (183.7, 156.4)
- moved D67 125.7 mm to (183.7, 160.4)
- moved D66 125.7 mm to (180.1, 160.4)
- moved D68 125.7 mm to (187.2, 160.4)
- moved COL10 84.8 mm to (256.3, 41.5)
- moved COL12 84.8 mm to (298.8, 40.3)
- moved COL4 84.8 mm to (145.6, 45.1)
- moved COL8 84.8 mm to (219.4, 42.7)
- moved COL11 84.8 mm to (274.7, 40.9)
- moved COL13 84.8 mm to (306.9, 40.0)
- moved COL5 84.8 mm to (164.0, 44.5)
- moved COL6 84.8 mm to (182.5, 43.9)
- moved COL7 84.8 mm to (200.9, 43.3)
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Routing:
- net /ROW4: track 7.50 -> 318.4 mm, vias 0 -> 2
- net /ROW3: track 0.00 -> 310.9 mm, vias 0 -> 2
- net /ROW0: track 0.00 -> 291.8 mm, vias 0 -> 2
- net /ROW2: track 0.00 -> 279.8 mm
- net /ROW1: track 0.00 -> 273.1 mm, vias 0 -> 2
- net /COL0: track 93.2 -> 148.8 mm
- net /COL12: track 122.8 -> 156.9 mm
- net Net-(D28-A): track 0.00 -> 30.5 mm
- net Net-(D29-A): track 0.00 -> 28.9 mm
- net Net-(D58-A): track 0.00 -> 28.4 mm
- net +3.3V: track 2.02 -> 30.1 mm
- net Net-(D59-A): track 16.7 -> 44.3 mm
- net Net-(D56-A): track 0.00 -> 25.2 mm
- net Net-(D57-A): track 0.00 -> 25.2 mm
- net Net-(D60-A): track 0.00 -> 25.2 mm
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
Commit message: wired up columns
Parts:
- J4: moved to F.Cu
- moved J4 30.0 mm to (113.2, 59.7), turned to 0 degrees
- moved U3 23.0 mm to (101.8, 62.3)
- moved J6 8.37 mm to (133.3, 85.0)
- moved C9 5.78 mm to (92.7, 106.0), turned to 180 degrees
- moved C3 5.78 mm to (92.7, 105.1), turned to 180 degrees
- moved C4 5.72 mm to (95.0, 110.9), turned to -90 degrees
- moved C6 5.56 mm to (101.5, 99.3), turned to 90 degrees
- moved C1 4.02 mm to (103.0, 109.9), turned to 0 degrees
- moved C2 3.05 mm to (102.1, 101.9), turned to 90 degrees
- moved J3 2.78 mm to (143.0, 107.7)
- moved U1 1.45 mm to (98.6, 106.4), turned to 0 degrees
- moved J1 0.54 mm to (96.4, 89.6)
Connections:
- U1 pad 10: /COL7 -> unconnected-(U1-PA0-Pad10)
- U1 pad 11: /COL6 -> unconnected-(U1-PA1-Pad11)
- U1 pad 12: /COL5 -> unconnected-(U1-PA2-Pad12)
- U1 pad 13: /COL4 -> unconnected-(U1-PA3-Pad13)
- U1 pad 2: /COL12 -> /COL4
- U1 pad 20: /COL0 -> unconnected-(U1-PB2-Pad20)
- U1 pad 3: /COL11 -> /COL3
- U1 pad 37: unconnected-(U1-PA14-Pad37) -> /COL13
- U1 pad 38: /COL2 -> /COL12
- U1 pad 39: /COL3 -> /COL11
- U1 pad 4: /COL10 -> /COL2
- U1 pad 40: unconnected-(U1-PB4-Pad40) -> /COL10
- U1 pad 41: unconnected-(U1-PB5-Pad41) -> /COL9
- U1 pad 42: unconnected-(U1-PB6-Pad42) -> /COL8
- U1 pad 43: unconnected-(U1-PB7-Pad43) -> /COL7
- U1 pad 45: /COL1 -> /COL6
- U1 pad 46: /COL13 -> /COL5
- U1 pad 5: /COL9 -> /COL1
- U1 pad 6: /COL8 -> /COL0
Routing:
- net /COL13: track 150.4 -> 379.0 mm
- net /COL12: track 156.9 -> 380.5 mm
- net /COL11: track 92.2 -> 290.3 mm
- net /COL10: track 77.6 -> 257.7 mm
- net /COL9: track 57.1 -> 218.6 mm
- net /COL8: track 64.2 -> 207.3 mm
- net /COL7: track 93.4 -> 218.3 mm
- net /COL6: track 109.0 -> 215.7 mm
- net /COL5: track 64.2 -> 152.6 mm
- net /COL4: track 64.5 -> 138.6 mm
- net /COL3: track 95.4 -> 152.2 mm
- net /ROW4: track 318.4 -> 273.5 mm, vias 2 -> 0
- net /ROW3: track 310.9 -> 270.3 mm, vias 2 -> 0
- net /COL2: track 95.6 -> 135.1 mm
- net /COL1: track 107.0 -> 132.6 mm
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