File: Uni60/UNI60_Hotswap/Uni60_Hotswap_KiCad/Uni60_Hotswap.kicad_sch (KiCad schematic)
At the start: 193 parts, among them J1 Conn_01x04, J2 Conn_01x04, J3 Conn_01x04, J4 Conn_01x04, J5 Conn_01x04, J6 Conn_01x04, J7 USB_C_Receptacle_USB2.0_14P, SW1 SW_Push, SW2 SW_Push, U1 STM32F072CBTx, U2 XC6206PxxxMR, U3 USBLC6-2SC6

Commit message: changed solder to hotswap sockets
Parts:
- removed KC_SPC_3U1, KC_SPLIT_SPC_3U1: MX_SW_solder, shentobento:SW_MX_1u, symbol shentobento:MX_SW_solder
- C1, C2, C3, C4, C5, C6, C7, C8, C9, R1: KiLib_Generator (none) -> SMD_2terminal_chip_molded
- J1, J2, J3, J4, J5, J6: KiLib_Generator (none) -> connector/SMD_single_row_plus_mounting_pad
- KC_0, KC_1, KC_2, KC_3, KC_4, KC_5, KC_6, KC_7, KC_8, KC_9, KC_<>1, KC_A1, KC_B1, KC_BKSP1, KC_BKSP2, KC_BSLS2, KC_BSLS_ISO1, KC_C1, KC_COMM1, KC_D1, KC_DOT1, KC_E1, KC_ENT1, KC_ENT_ISO1, KC_EQL1, KC_ESC1, KC_F1, KC_G1, KC_H1, KC_I1, KC_J1, KC_K1, KC_L1, KC_LBRC1, KC_LGUI1, KC_LSFT1, KC_M1, KC_MINS1, KC_MO1, KC_N1, KC_O1, KC_P1, KC_Q1, KC_QUOT1, KC_R1, KC_RBRC1, KC_RGUI1, KC_RSFT1, KC_RSFT_2.75u1, KC_S1, KC_SCLN1, KC_SLSH1, KC_SPC1, KC_SPC_2.75U1, KC_SPC_6.25U1, KC_SPLIT_SPC_2.25U1, KC_T1, KC_U1, KC_V1, KC_W1, KC_X1, KC_Y1, KC_Z1: footprint shentobento:SW_MX_1u -> shentobento:SW_MX_HS_KAILH_1u
- KC_BSLS1, KC_LALT1, KC_LCTL1, KC_RALT1, KC_RCTL1, KC_TAB1: footprint shentobento:SW_MX_1.5u -> shentobento:SW_MX_HS_KAILH_1.5u
- KC_CAPS1: footprint shentobento:SW_MX_1.75u -> shentobento:SW_MX_HS_KAILH_1.75u
- KC_LALT_1.25U1, KC_LCTL_1.25U1, KC_LGUI_1.25U1, KC_LSFT2, KC_MENU1, KC_RALT_1.25U1, KC_RCTL_1.25U1, KC_RGUI_1.25U1, KC_SPLIT_FN_1.25U1: footprint shentobento:SW_MX_1.25u -> shentobento:SW_MX_HS_KAILH_1.25u
- U1, U2, U3: KiLib_Generator (none) -> package/gullwing

Commit message: idk
Parts:
- D1, D10, D11, D12, D13, D14, D15, D16, D17, D18, D19, D2, D20, D21, D22, D23, D24, D25, D26, D27, D28, D29, D3, D30, D31, D32, D33, D34, D35, D36, D37, D38, D39, D4, D40, D41, D42, D43, D44, D45, D46, D47, D48, D49, D5, D50, D51, D52, D53, D54, D55, D56, D57, D58, D59, D6, D60, D61, D62, D63, D64, D65, D66, D67, D68, D69, D7, D70, D72, D73, D8, D9: footprint shentobento:D_SOD-123 -> Diode_SMD:D_SOD-323
- KC_STEP1: footprint shentobento:SW_MX_1.75u_STEPPED_1.25 -> shentobento:SW_MX_HS_KAILH_1.75u_STEPPED_1.25

Commit message: wired up columns
Connections:
- net COL0: now also U1.6 (PF1); no longer U1.20 (PB2)
- net COL1: now also U1.5 (PF0); no longer U1.45 (PB8)
- net COL10: now also U1.40 (PB4); no longer U1.4 (PC15)
- net COL11: now also U1.39 (PB3); no longer U1.3 (PC14)
- net COL12: now also U1.38 (PA15); no longer U1.2 (PC13)
- net COL13: now also U1.37 (PA14); no longer U1.46 (PB9)
- net COL2: now also U1.4 (PC15); no longer U1.38 (PA15)
- net COL3: now also U1.3 (PC14); no longer U1.39 (PB3)
- net COL4: now also U1.2 (PC13); no longer U1.13 (PA3)
- net COL5: now also U1.46 (PB9); no longer U1.12 (PA2)
- net COL6: now also U1.45 (PB8); no longer U1.11 (PA1)
- net COL7: now also U1.43 (PB7); no longer U1.10 (PA0)
- net COL8: now also U1.42 (PB6); no longer U1.6 (PF1)
- net COL9: now also U1.41 (PB5); no longer U1.5 (PF0)
Changed lines of the file:
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@@
 	)
 	(label "COL11"
-		(at 25.4 57.15 180)
+		(at 25.4 72.39 180)
 		(effects
 			(font
@@
 	)
 	(label "COL1"
-		(at 25.4 85.09 180)
+		(at 25.4 46.99 180)
 		(effects
 			(font
@@
 	)
 	(label "COL0"
-		(at 25.4 69.85 180)
+		(at 25.4 49.53 180)
 		(effects
 			(font
@@
 	)
 	(label "COL13"
-		(at 25.4 87.63 180)
+		(at 60.96 72.39 0)
 		(effects
 			(font
 				(size 1.27 1.27)
 			)
-			(justify right bottom)
+			(justify left bottom)
 		)
 	)
 	(label "COL6"
-		(at 60.96 39.37 0)
+		(at 25.4 85.09 180)
 		(effects
 			(font
 				(size 1.27 1.27)
 			)
-			(justify left bottom)
+			(justify right bottom)
 		)
 	)
@@
 	)
 	(label "COL8"
-		(at 25.4 49.53 180)
+		(at 25.4 80.01 180)
 		(effects
 			(font
@@
 	)
 	(label "COL7"
-		(at 60.96 36.83 0)
+		(at 25.4 82.55 180)
 		(effects
 			(font
 				(size 1.27 1.27)
 			)
-			(justify left bottom)
+			(justify right bottom)
 		)
 	)
 	(label "COL10"
-		(at 25.4 59.69 180)
+		(at 25.4 74.93 180)
 		(effects
 			(font
@@
 	)
 	(label "COL2"
-		(at 60.96 74.93 0)
+		(at 25.4 59.69 180)
 		(effects
 			(font
 				(size 1.27 1.27)
 			)
-			(justify left bottom)
+			(justify right bottom)
 		)
 	)
 	(label "COL3"
-		(at 25.4 72.39 180)
+		(at 25.4 57.15 180)
 		(effects
 			(font
@@
 	)
 	(label "COL5"
-		(at 60.96 41.91 0)
+		(at 25.4 87.63 180)
 		(effects
 			(font
 				(size 1.27 1.27)
 			)
-			(justify left bottom)
+			(justify right bottom)
 		)
 	)
@@
 	)
 	(label "COL9"
-		(at 25.4 46.99 180)
+		(at 25.4 77.47 180)
 		(effects
 			(font
@@
 	)
 	(label "COL12"
-		(at 25.4 54.61 180)
+		(at 60.96 74.93 0)
 		(effects
 			(font
 				(size 1.27 1.27)
 			)
-			(justify right bottom)
+			(justify left bottom)
 		)
 	)
@@
 	)
 	(label "COL4"
-		(at 60.96 44.45 0)
+		(at 25.4 54.61 180)
 		(effects
 			(font
 				(size 1.27 1.27)
 			)
-			(justify left bottom)
+			(justify right bottom)
 		)
 	)
@@
 		)
 	)
+	(group ""
+		(members "06e7def8-ba2f-44e9-ab62-5ffb9952b590" "09c15ece-6bf2-44fd-8e55-fb2ff4c52430"
+			"46c4e534-1cb2-4b96-867b-88eb1109e736" "77b679ae-e1e9-4230-9387-a0d23d8923e2"
+			"e48b57ec-2911-44a0-baa5-158ae35aa4e8" "eada93bc-4195-4ebc-a243-5775e06d322e"
+		)
+	)
